File: electrical/same54_dev_board/_autosave-USB_INTF.sch (KiCad schematic (older format))
At the start: 3 parts, among them J1 USB_B_Micro, U2 FT232RQ-REEL

Commit message: Trying to figure out how I want to do power...
Parts:
- added C?: 10nF, symbol Device:C_Small
- added FB?: 40_Ohm, symbol Device:Ferrite_Bead_Small
- gave numbers to parts that had none: 1
Connections:
- net GND: now also C?.2
- net g_5v: no longer J1.1 (VBUS), U2.19 (VCC)
- new net: C?.1, FB?.2, J1.1 (VBUS)
- new net: FB?.1, U2.19 (VCC)
Other:
- moved on the sheet: J1
Changed lines of the file:
@@
 L Connector:USB_B_Micro J1
 U 1 1 5E8480AD
-P 5050 3000
-F 0 "J1" H 5107 3467 50  0000 C CNN
-F 1 "USB_B_Micro" H 5107 3376 50  0000 C CNN
-F 2 "Connector_USB:USB_Micro-B_Wuerth_629105150521" H 5200 2950 50  0001 C CNN
-F 3 "~" H 5200 2950 50  0001 C CNN
-	1    5050 3000
+P 6050 1300
+F 0 "J1" H 6107 1767 50  0000 C CNN
+F 1 "USB_B_Micro" H 6107 1676 50  0000 C CNN
+F 2 "Connector_USB:USB_Micro-B_Wuerth_629105150521" H 6200 1250 50  0001 C CNN
+F 3 "~" H 6200 1250 50  0001 C CNN
+	1    6050 1300
 	1    0    0    -1
 $EndComp
@@
 Power Interface
 Wire Wire Line
-	5350 3000 5400 3000
-Text Label 5400 3000 0    50   ~ 0
+	6350 1300 6400 1300
+Text Label 6400 1300 0    50   ~ 0
 USB_D+
 Wire Wire Line
-	5350 3100 5400 3100
-Text Label 5400 3100 0    50   ~ 0
+	6350 1400 6400 1400
+Text Label 6400 1400 0    50   ~ 0
 USB_D-
 Wire Wire Line
@@
 	7500 4200 7500 4300
 $Comp
-L power:GND #PWR?
+L power:GND #PWR0110
 U 1 1 5E7B73F2
 P 7500 4300
-F 0 "#PWR?" H 7500 4050 50  0001 C CNN
+F 0 "#PWR0110" H 7500 4050 50  0001 C CNN
 F 1 "GND" H 7505 4127 50  0000 C CNN
 F 2 "" H 7500 4300 50  0001 C CNN
@@
 $EndComp
 Wire Wire Line
-	4950 3400 5050 3400
-Wire Wire Line
-	5050 3400 5050 3500
-Connection ~ 5050 3400
-$Comp
-L power:GND #PWR?
+	5950 1700 6050 1700
+Wire Wire Line
+	6050 1700 6050 1800
+Connection ~ 6050 1700
+$Comp
+L power:GND #PWR0111
 U 1 1 5E7BED3A
-P 5050 3500
-F 0 "#PWR?" H 5050 3250 50  0001 C CNN
-F 1 "GND" H 5055 3327 50  0000 C CNN
-F 2 "" H 5050 3500 50  0001 C CNN
-F 3 "" H 5050 3500 50  0001 C CNN
-	1    5050 3500
-	1    0    0    -1
-$EndComp
-Text Label 5350 2800 0    50   ~ 0
-5v
-NoConn ~ 5350 3200
+P 6050 1800
+F 0 "#PWR0111" H 6050 1550 50  0001 C CNN
+F 1 "GND" H 6055 1627 50  0000 C CNN
+F 2 "" H 6050 1800 50  0001 C CNN
+F 3 "" H 6050 1800 50  0001 C CNN
+	1    6050 1800
+	1    0    0    -1
+$EndComp
+NoConn ~ 6350 1500
 Wire Notes Line
 	600  600  2000 600
-Wire Wire Line
-	7600 2400 7600 2300
-Text Label 7600 2300 0    50   ~ 0
-5v
 Text Label 1350 1950 0    50   ~ 0
 FTDI_TX
@@
 	8000 2800 8500 2800
 $Comp
-L Device:C_Small C?
+L Device:C_Small C6
 U 1 1 5E7E8395
 P 8500 2900
-F 0 "C?" H 8592 2946 50  0000 L CNN
+F 0 "C6" H 8592 2946 50  0000 L CNN
 F 1 "100nF" H 8592 2855 50  0000 L CNN
 F 2 "" H 8500 2900 50  0001 C CNN
@@
 	8500 3000 8500 3100
 $Comp
-L power:GND #PWR?
+L power:GND #PWR0112
 U 1 1 5E7E91F3
 P 8500 3100
-F 0 "#PWR?" H 8500 2850 50  0001 C CNN
+F 0 "#PWR0112" H 8500 2850 50  0001 C CNN
 F 1 "GND" H 8505 2927 50  0000 C CNN
 F 2 "" H 8500 3100 50  0001 C CNN
@@
 	7700 4200 7800 4200
 Connection ~ 7700 4200
+$Comp
+L Device:C_Small C?
+U 1 1 5E7F85B7
+P 6800 1200
+F 0 "C?" H 6892 1246 50  0000 L CNN
+F 1 "10nF" H 6892 1155 50  0000 L CNN
+F 2 "" H 6800 1200 50  0001 C CNN
+F 3 "~" H 6800 1200 50  0001 C CNN
+	1    6800 1200
+	1    0    0    -1
+$EndComp
+Wire Wire Line
+	6350 1100 6800 1100
+Wire Wire Line
+	6800 1300 6800 1700
+Wire Wire Line
+	6800 1700 6050 1700
+Wire Wire Line
+	6800 1100 7050 1100
+Connection ~ 6800 1100
+$Comp
+L Device:Ferrite_Bead_Small FB?
+U 1 1 5E7FB1E4
+P 7150 1100
+F 0 "FB?" V 6913 1100 50  0000 C CNN
+F 1 "40_Ohm" V 7004 1100 50  0000 C CNN
+F 2 "" V 7080 1100 50  0001 C CNN
+F 3 "~" H 7150 1100 50  0001 C CNN
+	1    7150 1100
+	0    1    1    0
+$EndComp
+Wire Wire Line
+	7600 1100 7600 2400
+Wire Wire Line
+	7250 1100 7600 1100
 $EndSCHEMATC
