File: electrical/same54_dev_board/same54_dev_board.kicad_pcb (KiCad board)
At the start: 2 copper layers, 101.6 x 80 mm, 13 parts, among them J1 USB_B_Micro, J2 Conn_ARM_JTAG_SWD_10, J3 Conn_02x20_Odd_Even_LCD_INTF, J4 Barrel_Jack_Switch, Q1 Default PFET_A, Q2 Alt PFET_A, Q3 Default PFET_B, Q4 Alt PFET_B, U1 p_ATSAME54P20A-AU, U2 FT232RQ-REEL, U3 MAX7301AAX+, U4 NCP349MNAETBG, Y1 XOSC32

Commit message: migrating to laptop
Parts:
- moved U3 10.2 mm to (106.7, 77.5), turned to 0 degrees
- moved U1 3.81 mm to (90.2, 109.2)
Changed lines of the file:
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@@
   )
   (module proj_modules:SOP80P1030X264-36N (layer F.Cu)
-    (at 96.52 78.74 90)
-    (fp_text reference U3 (at -2.415 -8.587 90) (layer F.SilkS)
+    (at 106.68 77.47)
+    (fp_text reference U3 (at -2.415 -8.587) (layer F.SilkS)
       (effects (font (size 1 1) (thickness 0.015)))
     )
-    (fp_text value MAX7301AAX+ (at 5.84 8.587 90) (layer F.Fab)
+    (fp_text value MAX7301AAX+ (at 5.84 8.587) (layer F.Fab)
       (effects (font (size 1 1) (thickness 0.015)))
     )
@@
     (fp_circle (center -6.51 -7.34) (end -6.41 -7.34) (layer F.Fab) (width 0.2))
     (fp_circle (center -6.51 -7.34) (end -6.41 -7.34) (layer F.SilkS) (width 0.2))
-    (pad 36 smd rect (at 4.72 -6.8 90) (size 1.79 0.54) (layers F.Cu F.Paste F.Mask)
+    (pad 36 smd rect (at 4.72 -6.8) (size 1.79 0.54) (layers F.Cu F.Paste F.Mask)
       (net 122 g_3v3))
-    (pad 35 smd rect (at 4.72 -6 90) (size 1.79 0.54) (layers F.Cu F.Paste F.Mask)
+    (pad 35 smd rect (at 4.72 -6) (size 1.79 0.54) (layers F.Cu F.Paste F.Mask)
       (net 167 /s_SCREEN_INTF/~IO_EXPANDER_CS))
-    (pad 34 smd rect (at 4.72 -5.2 90) (size 1.79 0.54) (layers F.Cu F.Paste F.Mask)
+    (pad 34 smd rect (at 4.72 -5.2) (size 1.79 0.54) (layers F.Cu F.Paste F.Mask)
       (net 178 /MASTER_SPI_MOSI))
-    (pad 33 smd rect (at 4.72 -4.4 90) (size 1.79 0.54) (layers F.Cu F.Paste F.Mask)
+    (pad 33 smd rect (at 4.72 -4.4) (size 1.79 0.54) (layers F.Cu F.Paste F.Mask)
       (net 175 /MASTER_SPI_CLK))
-    (pad 32 smd rect (at 4.72 -3.6 90) (size 1.79 0.54) (layers F.Cu F.Paste F.Mask)
+    (pad 32 smd rect (at 4.72 -3.6) (size 1.79 0.54) (layers F.Cu F.Paste F.Mask)
       (net 123 "Net-(U3-Pad32)"))
-    (pad 31 smd rect (at 4.72 -2.8 90) (size 1.79 0.54) (layers F.Cu F.Paste F.Mask)
+    (pad 31 smd rect (at 4.72 -2.8) (size 1.79 0.54) (layers F.Cu F.Paste F.Mask)
       (net 124 "Net-(U3-Pad31)"))
-    (pad 30 smd rect (at 4.72 -2 90) (size 1.79 0.54) (layers F.Cu F.Paste F.Mask)
+    (pad 30 smd rect (at 4.72 -2) (size 1.79 0.54) (layers F.Cu F.Paste F.Mask)
       (net 125 "Net-(U3-Pad30)"))
-    (pad 29 smd rect (at 4.72 -1.2 90) (size 1.79 0.54) (layers F.Cu F.Paste F.Mask)
+    (pad 29 smd rect (at 4.72 -1.2) (size 1.79 0.54) (layers F.Cu F.Paste F.Mask)
       (net 126 "Net-(U3-Pad29)"))
-    (pad 28 smd rect (at 4.72 -0.4 90) (size 1.79 0.54) (layers F.Cu F.Paste F.Mask)
+    (pad 28 smd rect (at 4.72 -0.4) (size 1.79 0.54) (layers F.Cu F.Paste F.Mask)
       (net 137 /s_SCREEN_INTF/D23))
-    (pad 27 smd rect (at 4.72 0.4 90) (size 1.79 0.54) (layers F.Cu F.Paste F.Mask)
+    (pad 27 smd rect (at 4.72 0.4) (size 1.79 0.54) (layers F.Cu F.Paste F.Mask)
       (net 138 /s_SCREEN_INTF/D22))
-    (pad 26 smd rect (at 4.72 1.2 90) (size 1.79 0.54) (layers F.Cu F.Paste F.Mask)
+    (pad 26 smd rect (at 4.72 1.2) (size 1.79 0.54) (layers F.Cu F.Paste F.Mask)
       (net 139 /s_SCREEN_INTF/D21))
-    (pad 25 smd rect (at 4.72 2 90) (size 1.79 0.54) (layers F.Cu F.Paste F.Mask)
+    (pad 25 smd rect (at 4.72 2) (size 1.79 0.54) (layers F.Cu F.Paste F.Mask)
       (net 140 /s_SCREEN_INTF/D20))
-    (pad 24 smd rect (at 4.72 2.8 90) (size 1.79 0.54) (layers F.Cu F.Paste F.Mask)
+    (pad 24 smd rect (at 4.72 2.8) (size 1.79 0.54) (layers F.Cu F.Paste F.Mask)
       (net 141 /s_SCREEN_INTF/D19))
-    (pad 23 smd rect (at 4.72 3.6 90) (size 1.79 0.54) (layers F.Cu F.Paste F.Mask)
+    (pad 23 smd rect (at 4.72 3.6) (size 1.79 0.54) (layers F.Cu F.Paste F.Mask)
       (net 142 /s_SCREEN_INTF/D18))
-    (pad 22 smd rect (at 4.72 4.4 90) (size 1.79 0.54) (layers F.Cu F.Paste F.Mask)
+    (pad 22 smd rect (at 4.72 4.4) (size 1.79 0.54) (layers F.Cu F.Paste F.Mask)
       (net 143 /s_SCREEN_INTF/D17))
-    (pad 21 smd rect (at 4.72 5.2 90) (size 1.79 0.54) (layers F.Cu F.Paste F.Mask)
+    (pad 21 smd rect (at 4.72 5.2) (size 1.79 0.54) (layers F.Cu F.Paste F.Mask)
       (net 144 /s_SCREEN_INTF/D16))
-    (pad 20 smd rect (at 4.72 6 90) (size 1.79 0.54) (layers F.Cu F.Paste F.Mask)
+    (pad 20 smd rect (at 4.72 6) (size 1.79 0.54) (layers F.Cu F.Paste F.Mask)
       (net 145 /s_SCREEN_INTF/D15))
-    (pad 19 smd rect (at 4.72 6.8 90) (size 1.79 0.54) (layers F.Cu F.Paste F.Mask)
+    (pad 19 smd rect (at 4.72 6.8) (size 1.79 0.54) (layers F.Cu F.Paste F.Mask)
       (net 146 /s_SCREEN_INTF/D14))
-    (pad 18 smd rect (at -4.72 6.8 90) (size 1.79 0.54) (layers F.Cu F.Paste F.Mask)
+    (pad 18 smd rect (at -4.72 6.8) (size 1.79 0.54) (layers F.Cu F.Paste F.Mask)
       (net 147 /s_SCREEN_INTF/D13))
-    (pad 17 smd rect (at -4.72 6 90) (size 1.79 0.54) (layers F.Cu F.Paste F.Mask)
+    (pad 17 smd rect (at -4.72 6) (size 1.79 0.54) (layers F.Cu F.Paste F.Mask)
       (net 148 /s_SCREEN_INTF/D12))
-    (pad 16 smd rect (at -4.72 5.2 90) (size 1.79 0.54) (layers F.Cu F.Paste F.Mask)
+    (pad 16 smd rect (at -4.72 5.2) (size 1.79 0.54) (layers F.Cu F.Paste F.Mask)
       (net 149 /s_SCREEN_INTF/D11))
-    (pad 15 smd rect (at -4.72 4.4 90) (size 1.79 0.54) (layers F.Cu F.Paste F.Mask)
+    (pad 15 smd rect (at -4.72 4.4) (size 1.79 0.54) (layers F.Cu F.Paste F.Mask)
       (net 150 /s_SCREEN_INTF/D10))
-    (pad 14 smd rect (at -4.72 3.6 90) (size 1.79 0.54) (layers F.Cu F.Paste F.Mask)
+    (pad 14 smd rect (at -4.72 3.6) (size 1.79 0.54) (layers F.Cu F.Paste F.Mask)
       (net 151 /s_SCREEN_INTF/D9))
-    (pad 13 smd rect (at -4.72 2.8 90) (size 1.79 0.54) (layers F.Cu F.Paste F.Mask)
+    (pad 13 smd rect (at -4.72 2.8) (size 1.79 0.54) (layers F.Cu F.Paste F.Mask)
       (net 152 /s_SCREEN_INTF/D8))
-    (pad 12 smd rect (at -4.72 2 90) (size 1.79 0.54) (layers F.Cu F.Paste F.Mask)
+    (pad 12 smd rect (at -4.72 2) (size 1.79 0.54) (layers F.Cu F.Paste F.Mask)
       (net 153 /s_SCREEN_INTF/D7))
-    (pad 11 smd rect (at -4.72 1.2 90) (size 1.79 0.54) (layers F.Cu F.Paste F.Mask)
+    (pad 11 smd rect (at -4.72 1.2) (size 1.79 0.54) (layers F.Cu F.Paste F.Mask)
       (net 154 /s_SCREEN_INTF/D6))
-    (pad 10 smd rect (at -4.72 0.4 90) (size 1.79 0.54) (layers F.Cu F.Paste F.Mask)
+    (pad 10 smd rect (at -4.72 0.4) (size 1.79 0.54) (layers F.Cu F.Paste F.Mask)
       (net 155 /s_SCREEN_INTF/D5))
-    (pad 9 smd rect (at -4.72 -0.4 90) (size 1.79 0.54) (layers F.Cu F.Paste F.Mask)
+    (pad 9 smd rect (at -4.72 -0.4) (size 1.79 0.54) (layers F.Cu F.Paste F.Mask)
       (net 156 /s_SCREEN_INTF/D4))
-    (pad 8 smd rect (at -4.72 -1.2 90) (size 1.79 0.54) (layers F.Cu F.Paste F.Mask)
+    (pad 8 smd rect (at -4.72 -1.2) (size 1.79 0.54) (layers F.Cu F.Paste F.Mask)
       (net 157 /s_SCREEN_INTF/D3))
-    (pad 7 smd rect (at -4.72 -2 90) (size 1.79 0.54) (layers F.Cu F.Paste F.Mask)
+    (pad 7 smd rect (at -4.72 -2) (size 1.79 0.54) (layers F.Cu F.Paste F.Mask)
       (net 158 /s_SCREEN_INTF/D2))
-    (pad 6 smd rect (at -4.72 -2.8 90) (size 1.79 0.54) (layers F.Cu F.Paste F.Mask)
+    (pad 6 smd rect (at -4.72 -2.8) (size 1.79 0.54) (layers F.Cu F.Paste F.Mask)
       (net 159 /s_SCREEN_INTF/D1))
-    (pad 5 smd rect (at -4.72 -3.6 90) (size 1.79 0.54) (layers F.Cu F.Paste F.Mask)
+    (pad 5 smd rect (at -4.72 -3.6) (size 1.79 0.54) (layers F.Cu F.Paste F.Mask)
       (net 160 /s_SCREEN_INTF/D0))
-    (pad 4 smd rect (at -4.72 -4.4 90) (size 1.79 0.54) (layers F.Cu F.Paste F.Mask)
+    (pad 4 smd rect (at -4.72 -4.4) (size 1.79 0.54) (layers F.Cu F.Paste F.Mask)
       (net 174 /MASTER_SPI_MISO))
-    (pad 3 smd rect (at -4.72 -5.2 90) (size 1.79 0.54) (layers F.Cu F.Paste F.Mask)
+    (pad 3 smd rect (at -4.72 -5.2) (size 1.79 0.54) (layers F.Cu F.Paste F.Mask)
       (net 127 GND))
-    (pad 2 smd rect (at -4.72 -6 90) (size 1.79 0.54) (layers F.Cu F.Paste F.Mask)
+    (pad 2 smd rect (at -4.72 -6) (size 1.79 0.54) (layers F.Cu F.Paste F.Mask)
       (net 127 GND))
-    (pad 1 smd rect (at -4.72 -6.8 90) (size 1.79 0.54) (layers F.Cu F.Paste F.Mask)
+    (pad 1 smd rect (at -4.72 -6.8) (size 1.79 0.54) (layers F.Cu F.Paste F.Mask)
       (net 128 "Net-(R1-Pad1)"))
   )
@@
   )
   (module penguin:QFP40P1600X1600X120-128N_ATSAME54P20A (layer F.Cu)
-    (at 86.36 109.22 45)
+    (at 90.17 109.22 45)
     (fp_text reference U1 (at -4.500975 -9.803025 45) (layer F.SilkS)
       (effects (font (size 1.001331 1.001331) (thickness 0.015)))
