File: electrical/2x20_breakout_board/breakout_board_2x20/breakout_board_2x20.kicad_pcb (KiCad board)
At the start: 2 copper layers, 66 x 69.8 mm, 2 parts, among them J1 Conn_02x20_Odd_Even, J2 Conn_02x20_Odd_Even_LCD_INTF

Commit message: .
Other:
- board text added: "Mikro 4" TFT Breakout"
Changed lines of the file:
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@@
   (general
     (thickness 1.6)
-    (drawings 10)
+    (drawings 11)
     (tracks 720)
     (zones 0)
@@
     (visible_elements 7FFFFFFF)
     (pcbplotparams
-      (layerselection 0x010fc_ffffffff)
-      (usegerberextensions false)
+      (layerselection 0x010f0_ffffffff)
+      (usegerberextensions true)
       (usegerberattributes false)
       (usegerberadvancedattributes false)
@@
       (psa4output false)
       (plotreference true)
-      (plotvalue true)
+      (plotvalue false)
       (plotinvisibletext false)
-      (padsonsilk false)
+      (padsonsilk true)
       (subtractmaskfromsilk false)
       (outputformat 1)
       (mirror false)
-      (drillshape 1)
+      (drillshape 0)
       (scaleselection 1)
-      (outputdirectory ""))
+      (outputdirectory "gerbers/"))
   )
   (net 0 "")
@@
     )
   )
+  (gr_text "Mikro 4\" TFT Breakout" (at 154.686 32.258) (layer B.SilkS)
+    (effects (font (size 1 1) (thickness 0.15)) (justify mirror))
+  )
   (gr_line (start 143.51 100.33) (end 143.51 96.52) (layer Edge.Cuts) (width 0.05))
